File: minister.kicad_pcb (KiCad board)
At the start: 2 copper layers, 108 parts, among them SW1 SW_Push, U1 ATmega32U4-AU, Y1 16MHz

Commit message: move surface mount componets to bottom with 'F'
Parts:
- C1, C2, C3, C4, C5, C6, C7, D1, D10, D11, D12, D13, D14, D15, D16, D17, D18, D19, D2, D20, D21, D22, D23, D24, D25, D26, D27, D28, D29, D3, D30, D31, D32, D33, D34, D35, D36, D37, D38, D39, D4, D40, D41, D42, D43, D44, D45, D46, D5, D6, D7, D8, D9, F1, R1, R2, R3, R4, SW1, U1, USB1, Y1: moved to B.Cu
- moved R2 15.3 mm to (138.3, 65.9)
- moved D6 15.1 mm to (84.9, 81.8)
- moved R3 14.1 mm to (138.0, 71.4)
- moved D43 7.18 mm to (212.7, 176.2)
- moved D5 6.29 mm to (56.4, 81.8)
- moved D14 4.83 mm to (-42.1, 116.7)
- moved D44 4.57 mm to (255.5, 176.2)

Commit message: import prime_e edge cuts
Parts:
- C7: value 0.1uF -> 10uF
- MX42: footprint MX_Only:MXOnly-2U-Hotswap -> MX_Only:MXOnly-2U-Hotswap-ReversedStabilizers
- MX43: footprint MX_Only:MXOnly-2.25U-Hotswap -> MX_Only:MXOnly-2.25U-Hotswap-ReversedStabilizers
- moved C2 193.7 mm to (126.6, -71.5), turned to 270 degrees
- moved C1 187.7 mm to (136.7, -71.5), turned to 90 degrees
- moved Y1 187.6 mm to (131.8, -71.5), turned to 180 degrees
- moved R1 183.2 mm to (128.0, -38.7), turned to 270 degrees
- moved SW1 176.6 mm to (124.8, -29.0), turned to 180 degrees
- moved R3 175.3 mm to (126.4, -103.5), turned to 90 degrees
- moved C5 164.1 mm to (108.7, -62.5), turned to 270 degrees
- moved C4 163.4 mm to (113.5, -62.5), turned to 270 degrees
- moved R2 163.3 mm to (128.8, -97.1), turned to 90 degrees
- moved C3 161.9 mm to (113.0, -56.4), turned to 270 degrees
- moved D26 160.4 mm to (-56.9, -13.1), turned to 90 degrees
- moved D27 159.9 mm to (-26.8, -13.1), turned to 90 degrees
- moved C7 159.0 mm to (99.2, -62.5), turned to 270 degrees
- moved C6 158.8 mm to (103.9, -62.5), turned to 270 degrees
- moved D1 158.6 mm to (-59.3, -74.3), turned to 90 degrees
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Other:
- board outline added: 276.7 x 91.9 mm

Commit message: everything laid out
Parts:
- moved USB1 187.7 mm to (138.3, 66.3)
- moved MX1 186.3 mm to (23.6, 76.6)
- moved F1 185.7 mm to (135.5, 76.7)
- moved C7 185.7 mm to (140.8, 118.5), turned to 90 degrees
- moved C4 183.9 mm to (146.2, 118.5)
- moved MX5 183.7 mm to (100.3, 82.3), turned to 352 degrees
- moved MX6 183.2 mm to (119.3, 85.0), turned to 352 degrees
- moved MX4 183.2 mm to (81.4, 79.6), turned to 352 degrees
- moved MX2 182.4 mm to (42.7, 76.6)
- moved MX3 181.6 mm to (62.6, 77.0), turned to 352 degrees
- moved MX7 180.1 mm to (157.7, 86.2), turned to 8 degrees
- moved R3 180.0 mm to (138.2, 76.1)
- moved D1 179.9 mm to (32.1, 80.6)
- moved R4 179.4 mm to (143.5, 118.5), turned to 90 degrees
- moved D5 177.9 mm to (108.1, 87.9), turned to 82 degrees
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Other:
- outline, holes or cut-outs redrawn

Commit message: use shaped edge cuts
Parts:
- moved D38 2.39 mm to (281.7, 119.4)
- moved R2 0.66 mm to (141.2, 76.5)
- moved R3 0.41 mm to (138.2, 76.5)
- moved F1 0.36 mm to (135.3, 76.5)
Other:
- board size 276.7 x 91.9 mm -> 271.5 x 90.5 mm

Commit message: start routing
Parts:
- moved C7 22.1 mm to (149.8, 98.3), turned to 180 degrees
- moved C5 18.8 mm to (140.7, 118.6), turned to 270 degrees
- moved C3 6.27 mm to (133.3, 113.7)
- moved C6 5.76 mm to (133.3, 110.9)
- moved C4 2.67 mm to (143.5, 118.4)
- moved R4 2.67 mm to (146.2, 118.4)
- moved R1 1.14 mm to (134.7, 104.1)
- moved R2 1.14 mm to (140.1, 76.5)
- moved D19 0.95 mm to (128.2, 109.8)
- moved D38 0.77 mm to (282.4, 119.5)
- moved MX42 0.25 mm to (116.0, 142.2)
- moved R3 0.25 mm to (137.9, 76.5)
- moved F1 0.13 mm to (135.1, 76.5)
- moved MX43 0.13 mm to (172.7, 142.0)
Routing:
- net ROW1: track 0.00 -> 298.4 mm, vias 0 -> 12
- net ROW2: track 0.00 -> 297.4 mm, vias 0 -> 13
- net ROW0: track 0.00 -> 294.9 mm, vias 0 -> 13
- net ROW3: track 0.00 -> 257.5 mm
- net COL0: track 0.00 -> 174.8 mm, vias 0 -> 1
- net COL12: track 0.00 -> 167.1 mm, vias 0 -> 1
- net COL1: track 0.00 -> 159.9 mm, vias 0 -> 1
- net COL11: track 0.00 -> 154.1 mm, vias 0 -> 1
- net COL3: track 0.00 -> 124.4 mm, vias 0 -> 1
- net COL2: track 0.00 -> 119.7 mm, vias 0 -> 1
- net +5V: track 0.00 -> 118.2 mm, vias 0 -> 5
- net COL10: track 0.00 -> 111.6 mm, vias 0 -> 1
- net COL4: track 0.00 -> 107.8 mm, vias 0 -> 1
- net COL8: track 0.00 -> 101.6 mm, vias 0 -> 1
- net COL9: track 0.00 -> 97.4 mm, vias 0 -> 1
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Other:
- outline, holes or cut-outs redrawn
- net class Power added: clearance 0.2, trace_width 0.381, via_dia 0.8, via_drill 0.4

Commit message: more routing
Parts:
- moved F1 6.86 mm to (136.4, 83.2)
- moved R3 6.14 mm to (138.7, 82.6)
- moved R2 6.13 mm to (140.7, 82.6)
- moved USB1 2.13 mm to (138.9, 68.3)
Connections:
- U1 pad 1: Net-(U1-Pad1) -> ROW0
- U1 pad 18: Net-(U1-Pad18) -> COL12
- U1 pad 19: Net-(U1-Pad19) -> COL11
- U1 pad 20: Net-(U1-Pad20) -> COL10
- U1 pad 21: Net-(U1-Pad21) -> COL9
- U1 pad 22: Net-(U1-Pad22) -> COL8
- U1 pad 25: Net-(U1-Pad25) -> COL7
- U1 pad 26: Net-(U1-Pad26) -> COL6
- U1 pad 28: Net-(U1-Pad28) -> ROW3
- U1 pad 29: Net-(U1-Pad29) -> ROW2
- U1 pad 32: Net-(U1-Pad32) -> ROW1
- U1 pad 36: Net-(U1-Pad36) -> COL5
- U1 pad 37: Net-(U1-Pad37) -> COL4
- U1 pad 38: Net-(U1-Pad38) -> COL3
- U1 pad 39: Net-(U1-Pad39) -> COL2
- U1 pad 40: Net-(U1-Pad40) -> COL1
- U1 pad 41: Net-(U1-Pad41) -> COL0
Routing:
- net +5V: track 118.2 -> 111.6 mm, vias 5 -> 6
- net Net-(R2-Pad1): track 34.1 -> 28.2 mm
- net Net-(R3-Pad1): track 34.3 -> 28.5 mm
- net VCC: track 4.91 -> 9.35 mm
- net D-: track 4.97 -> 9.09 mm
- net D+: track 5.51 -> 9.57 mm
Other:
- board size 271.5 x 90.5 mm -> 271.5 x 88.5 mm

Commit message: all routing done? except for gnd
Parts:
- moved R1 15.5 mm to (148.7, 97.5), turned to 90 degrees
- moved C7 1.91 mm to (151.7, 98.2), turned to 0 degrees
- moved C4 1.05 mm to (143.5, 119.5)
- moved R4 1.05 mm to (146.2, 119.5)
- moved U1 0.90 mm to (144.3, 106.7), turned to 315 degrees
Routing:
- net ROW3: track 257.5 -> 315.5 mm, vias 0 -> 8
- net COL7: track 57.2 -> 81.6 mm, vias 1 -> 2
- net ROW2: track 297.4 -> 321.2 mm, vias 13 -> 14
- net COL11: track 154.1 -> 175.3 mm, vias 1 -> 2
- net COL12: track 167.1 -> 188.2 mm, vias 1 -> 2
- net COL10: track 111.6 -> 132.3 mm, vias 1 -> 2
- net COL9: track 97.4 -> 117.9 mm, vias 1 -> 2
- net COL8: track 101.6 -> 122.0 mm, vias 1 -> 2
- net ROW0: track 294.9 -> 311.6 mm, vias 13 -> 14
- net COL5: track 61.1 -> 76.9 mm, vias 1 -> 2
- net Net-(C3-Pad1): track 0.00 -> 15.6 mm
- net COL2: track 119.7 -> 134.7 mm, vias 1 -> 2
- net COL0: track 174.8 -> 189.6 mm, vias 1 -> 2
- net COL3: track 124.4 -> 138.5 mm, vias 1 -> 2
- net COL1: track 159.9 -> 173.4 mm, vias 1 -> 2
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Other:
- board size 271.5 x 88.5 mm -> 271.5 x 88.1 mm

Commit message: add ground fill and run drc
Parts:
- turned C3 to 0 degrees
Routing:
- net GND: track 5.46 -> 113.4 mm, vias 0 -> 11
- net Net-(C3-Pad1): track 15.6 -> 19.3 mm
- net COL7: track 81.6 -> 84.3 mm
- net +5V: track 108.6 -> 111.0 mm, vias 6 -> 8
- net Net-(R2-Pad1): track 22.5 -> 23.9 mm
- net COL2: track 134.7 -> 133.8 mm
- net ROW3: track 315.5 -> 316.3 mm, vias 8 -> 9
- net Net-(R3-Pad1): track 22.4 -> 23.0 mm
- net COL1: track 173.4 -> 172.9 mm
- added copper zone on B.Cu, net GND
- added copper zone on F.Cu, net GND
Other:
- board text added: "BY MAKENOVA"
- board text added: "MINISTER_E V0"
