File: minister.sch (KiCad schematic (older format))
At the start: 112 parts, among them J1 AVR-ISP-6, SW1 SW_Push, U1 ATmega32U4-AU, Y1 16MHz

Commit message: submit for production
generate gerbers and drill files
generate bom and placement file
update some parts
Parts:
- C1, C2: Field4 C1804 -> (none); LCSC (none) -> C1804
- C3: Field4 C28323 -> (none); LCSC (none) -> C28323
- C4, C5, C6: Field4 C49678 -> (none); LCSC (none) -> C49678
- C7: Field4 C307523 -> (none); LCSC (none) -> C307523
- D1, D10, D11, D12, D13, D14, D15, D16, D17, D18, D19, D2, D20, D21, D22, D23, D24, D25, D26, D27, D28, D29, D3, D30, D31, D32, D33, D34, D35, D36, D37, D38, D39, D4, D40, D41, D42, D43, D44, D45, D46, D5, D6, D7, D8, D9: Field4 C81598 -> (none); LCSC (none) -> C81598
- D47: Field4 C78442 -> (none); LCSC (none) -> C78442
- F1: Field4 C151162 -> (none); LCSC (none) -> C151162
- R1, R4: Field4 C17414 -> (none); LCSC (none) -> C17414
- R5, R8: Field4 C27834 -> (none); LCSC (none) -> C27834
- R6, R7: Field4 C17561 -> (none); LCSC (none) -> C17561
- SW1: Field4 C318884 -> (none); LCSC (none) -> C318884
- U1: LCSC (none) -> C44854
- Y1: Field4 C89379 -> (none); LCSC (none) -> C89379
